File: saiph_rev2/saiph_rev2.kicad_sch (KiCad schematic)
At the start: 209 parts, among them J1 USB_mini_micro_B, SW1 SW_PUSH, SW10 SW_PUSH, SW100 SW_PUSH, SW101 SW_PUSH, SW102 SW_PUSH, SW103 SW_PUSH, SW104 SW_PUSH, SW105 SW_PUSH, SW108 SKQGABE010, SW109 SW_PUSH, SW11 SW_PUSH, SW110 SW_PUSH, SW111 SW_PUSH, SW112 SKQGABE010, SW12 SW_PUSH, SW13 SW_PUSH, SW14 SW_PUSH, SW15 SW_PUSH, SW16 SW_PUSH, SW17 SW_PUSH, SW18 SW_PUSH, SW19 SW_PUSH, SW2 SW_PUSH, SW20 SW_PUSH, SW21 SW_PUSH, SW22 SW_PUSH, SW23 SW_PUSH, SW24 SW_PUSH, SW25 SW_PUSH, SW26 SW_PUSH, SW27 SW_PUSH, SW28 SW_PUSH, SW29 SW_PUSH, SW3 SW_PUSH, SW30 SW_PUSH, SW31 SW_PUSH, SW32 SW_PUSH, SW33 SW_PUSH, SW34 SW_PUSH, SW35 SW_PUSH, SW36 SW_PUSH, SW37 SW_PUSH, SW38 SW_PUSH, SW39 SW_PUSH, SW4 SW_PUSH, SW40 SW_PUSH, SW41 SW_PUSH, SW42 SW_PUSH, SW43 SW_PUSH, SW44 SW_PUSH, SW45 SW_PUSH, SW46 SW_PUSH, SW47 SW_PUSH, SW48 SW_PUSH, SW49 SW_PUSH, SW5 SW_PUSH, SW50 SW_PUSH, SW51 SW_PUSH, SW52 SW_PUSH, SW53 SW_PUSH, SW54 SW_PUSH, SW55 SW_PUSH, SW56 SW_PUSH, SW57 SW_PUSH, SW58 SW_PUSH, SW59 SW_PUSH, SW6 SW_PUSH, SW60 SW_PUSH, SW61 SW_PUSH, SW62 SW_PUSH, SW63 SW_PUSH, SW64 SW_PUSH, SW65 SW_PUSH, SW66 SW_PUSH, SW67 SW_PUSH, SW68 SW_PUSH, SW69 SW_PUSH, SW7 SW_PUSH, SW70 SW_PUSH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

Commit message: route more diodes
Connections:
- net C5: now also SW62.1, SW66.1
- net C6: no longer SW62.1, SW66.1
- net R4: now also D62.2 (A); no longer D62.1 (K)
- net at SW62.2, SW66.2: now also D62.1 (K); no longer D62.2 (A)
Other:
- moved on the sheet: D62, SW62, SW66
Changed lines of the file:
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@@
   (junction (at 417.83 129.54) (diameter 0) (color 0 0 0 0)
   )
+  (junction (at 392.43 109.22) (diameter 0) (color 0 0 0 0)
+  )
   (junction (at 280.67 129.54) (diameter 0) (color 0 0 0 0)
   )
@@
   (junction (at 128.27 116.84) (diameter 0) (color 0 0 0 0)
   )
-  (junction (at 415.29 109.22) (diameter 0) (color 0 0 0 0)
-  )
   (junction (at 306.07 63.5) (diameter 0) (color 0 0 0 0)
   )
@@
   (junction (at 237.49 73.66) (diameter 0) (color 0 0 0 0)
   )
-  (junction (at 417.83 109.22) (diameter 0) (color 0 0 0 0)
-  )
   (junction (at 410.21 134.62) (diameter 0) (color 0 0 0 0)
   )
@@
   (junction (at 135.89 55.88) (diameter 0) (color 0 0 0 0)
   )
-  (junction (at 435.61 116.84) (diameter 0) (color 0 0 0 0)
-  )
   (junction (at 128.27 127) (diameter 0) (color 0 0 0 0)
   )
@@
   (junction (at 135.89 109.22) (diameter 0) (color 0 0 0 0)
   )
+  (junction (at 389.89 109.22) (diameter 0) (color 0 0 0 0)
+  )
   (junction (at 491.49 109.22) (diameter 0) (color 0 0 0 0)
   )
@@
   (junction (at 433.07 81.28) (diameter 0) (color 0 0 0 0)
   )
-  (junction (at 433.07 109.22) (diameter 0) (color 0 0 0 0)
+  (junction (at 407.67 109.22) (diameter 0) (color 0 0 0 0)
   )
   (junction (at 288.29 73.66) (diameter 0) (color 0 0 0 0)
@@
   (junction (at 491.49 38.1) (diameter 0) (color 0 0 0 0)
   )
+  (junction (at 410.21 116.84) (diameter 0) (color 0 0 0 0)
+  )
   (junction (at 255.27 63.5) (diameter 0) (color 0 0 0 0)
   )
@@
     (stroke (width 0) (type default))
   )
-  (wire (pts (xy 389.89 91.44) (xy 389.89 127))
+  (wire (pts (xy 389.89 91.44) (xy 389.89 109.22))
     (stroke (width 0) (type default))
   )
@@
     (stroke (width 0) (type default))
   )
+  (wire (pts (xy 410.21 116.84) (xy 483.87 116.84))
+    (stroke (width 0) (type default))
+  )
   (wire (pts (xy 534.67 63.5) (xy 560.07 63.5))
     (stroke (width 0) (type default))
@@
     (stroke (width 0) (type default))
   )
-  (wire (pts (xy 435.61 116.84) (xy 483.87 116.84))
-    (stroke (width 0) (type default))
-  )
   (wire (pts (xy 509.27 63.5) (xy 534.67 63.5))
     (stroke (width 0) (type default))
@@
     (stroke (width 0) (type default))
   )
+  (wire (pts (xy 389.89 109.22) (xy 389.89 127))
+    (stroke (width 0) (type default))
+  )
   (wire (pts (xy 255.27 45.72) (xy 306.07 45.72))
     (stroke (width 0) (type default))
@@
     (stroke (width 0) (type default))
   )
+  (wire (pts (xy 389.89 109.22) (xy 392.43 109.22))
+    (stroke (width 0) (type default))
+  )
   (wire (pts (xy 339.09 55.88) (xy 339.09 73.66))
     (stroke (width 0) (type default))
@@
     (stroke (width 0) (type default))
   )
-  (wire (pts (xy 417.83 109.22) (xy 417.83 115.57))
+  (wire (pts (xy 392.43 109.22) (xy 392.43 115.57))
     (stroke (width 0) (type default))
   )
@@
     (stroke (width 0) (type default))
   )
-  (wire (pts (xy 433.07 109.22) (xy 433.07 115.57))
+  (wire (pts (xy 407.67 109.22) (xy 407.67 115.57))
     (stroke (width 0) (type default))
   )
@@
     (stroke (width 0) (type default))
   )
-  (wire (pts (xy 382.27 116.84) (xy 435.61 116.84))
+  (wire (pts (xy 382.27 116.84) (xy 410.21 116.84))
     (stroke (width 0) (type default))
   )
@@
     (stroke (width 0) (type default))
   )
-  (wire (pts (xy 415.29 109.22) (xy 415.29 127))
-    (stroke (width 0) (type default))
-  )
   (wire (pts (xy 441.96 55.88) (xy 441.96 60.96))
     (stroke (width 0) (type default))
@@
     (stroke (width 0) (type default))
   )
-  (wire (pts (xy 415.29 109.22) (xy 417.83 109.22))
-    (stroke (width 0) (type default))
-  )
   (wire (pts (xy 161.29 127) (xy 163.83 127))
     (stroke (width 0) (type default))
@@
     (stroke (width 0) (type default))
   )
-  (wire (pts (xy 415.29 91.44) (xy 415.29 109.22))
+  (wire (pts (xy 415.29 91.44) (xy 415.29 127))
     (stroke (width 0) (type default))
   )
@@
     (stroke (width 0) (type default))
   )
-  (wire (pts (xy 433.07 109.22) (xy 435.61 109.22))
+  (wire (pts (xy 407.67 109.22) (xy 410.21 109.22))
     (stroke (width 0) (type default))
   )
@@
     (effects (font (size 1.27 1.27)) (justify left bottom))
   )
-  (text "SHIFT" (at 433.07 106.68 0)
+  (text "SHIFT" (at 407.67 106.68 0)
     (effects (font (size 1.27 1.27)) (justify left bottom))
   )
@@
     )
   )
-  (symbol (lib_id "keyboard_parts:SW_PUSH") (at 425.45 115.57 0) (unit 1)
+  (symbol (lib_id "keyboard_parts:SW_PUSH") (at 400.05 115.57 0) (unit 1)
     (in_bom yes) (on_board yes) (dnp no)
-    (property "Reference" "SW66" (at 429.26 112.776 0)
+    (property "Reference" "SW66" (at 403.86 112.776 0)
       (effects (font (size 1.27 1.27)))
     )
-    (property "Value" "SW_PUSH" (at 425.45 117.602 0)
+    (property "Value" "SW_PUSH" (at 400.05 117.602 0)
       (effects (font (size 1.27 1.27)))
     )
-    (property "Footprint" "keyboard_parts:ALPS_PLATE" (at 425.45 115.57 0)
+    (property "Footprint" "keyboard_parts:ALPS_PLATE" (at 400.05 115.57 0)
       (effects (font (size 1.27 1.27)) hide)
     )
-    (property "Datasheet" "" (at 425.45 115.57 0)
+    (property "Datasheet" "" (at 400.05 115.57 0)
       (effects (font (size 1.27 1.27)))
     )
@@
     )
   )
-  (symbol (lib_id "keyboard_parts:SW_PUSH") (at 425.45 109.22 0) (unit 1)
+  (symbol (lib_id "keyboard_parts:SW_PUSH") (at 400.05 109.22 0) (unit 1)
     (in_bom yes) (on_board yes) (dnp no)
-    (property "Reference" "SW62" (at 429.26 106.426 0)
+    (property "Reference" "SW62" (at 403.86 106.426 0)
       (effects (font (size 1.27 1.27)))
     )
-    (property "Value" "SW_PUSH" (at 425.45 111.252 0)
+    (property "Value" "SW_PUSH" (at 400.05 111.252 0)
       (effects (font (size 1.27 1.27)))
     )
-    (property "Footprint" "keyboard_parts:ALPS_PLATE" (at 425.45 109.22 0)
+    (property "Footprint" "keyboard_parts:ALPS_PLATE" (at 400.05 109.22 0)
       (effects (font (size 1.27 1.27)) hide)
     )
-    (property "Datasheet" "" (at 425.45 109.22 0)
+    (property "Datasheet" "" (at 400.05 109.22 0)
       (effects (font (size 1.27 1.27)))
     )
@@
     )
   )
-  (symbol (lib_id "Diode:1N4148") (at 435.61 113.03 90) (unit 1)
+  (symbol (lib_id "Diode:1N4148") (at 410.21 113.03 270) (unit 1)
     (in_bom yes) (on_board yes) (dnp no)
-    (property "Reference" "D62" (at 433.07 113.03 0)
+    (property "Reference" "D62" (at 412.75 113.03 0)
       (effects (font (size 1.27 1.27)))
     )
-    (property "Value" "D" (at 438.15 113.03 0)
+    (property "Value" "D" (at 407.67 113.03 0)
       (effects (font (size 1.27 1.27)))
     )
-    (property "Footprint" "Diodes_ThroughHole:D_DO-35_SOD27_P7.62mm_Horizontal" (at 435.61 113.03 0)
+    (property "Footprint" "Diodes_ThroughHole:D_DO-35_SOD27_P7.62mm_Horizontal" (at 410.21 113.03 0)
       (effects (font (size 1.27 1.27)) hide)
     )
-    (property "Datasheet" "" (at 435.61 113.03 0)
+    (property "Datasheet" "" (at 410.21 113.03 0)
       (effects (font (size 1.27 1.27)))
     )

Commit message: routing pretty much done.
Connections:
- net C8: now also U1.21 (GPIO20); no longer U1.9 (GPIO8)
Changed lines of the file:
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@@
-    (effects (font (size 1.524 1.524)) (justify left))
-  )
-  (hierarchical_label "C8" (shape input) (at 143.51 191.77 0) (fields_autoplaced)
     (effects (font (size 1.524 1.524)) (justify left))
   )
@@
     (effects (font (size 1.524 1.524)) (justify left))
   )
+  (hierarchical_label "C8" (shape input) (at 143.51 222.25 0) (fields_autoplaced)
+    (effects (font (size 1.524 1.524)) (justify left))
+  )
